File: 1.pcb/openpci2-backplane/RC_4-lines-PCIe.kicad_sch (KiCad schematic)
At the start: 30 parts, among them J2 PCIE-064-02-X-D-TH, J3 1-2199230-6, J4 525591652, U7 TPS563206DRLR, X1 39-28-1063

Commit message: Replaced Clock generator
Parts:
- C48: DigiKey 399-3683-1-ND -> PCE4579CT-ND; Mouser 80-T491A106K0067280 -> 667-EEE-1CA101WAP; TME T491A106K006AT -> EEE1CA101WAP
- D2: Uvitron n/a -> (none)
- JP9: value ~ -> n/a
- renumbered R16 to R14, R17 to R15, R18 to R16, R19 to R17, R20 to R18, R21 to R19, U7 to U6
Other:
- note added: "Decide where to connect +3.3Vaux!"
Changed lines of the file:
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@@
 		)
 	)
+	(text "Decide where to connect +3.3Vaux!"
+		(exclude_from_sim no)
+		(at 95.758 86.106 0)
+		(effects
+			(font
+				(size 1.27 1.27)
+				(color 255 0 0 1)
+			)
+		)
+	)
 	(text "One high power down converter or one per slot?"
 		(exclude_from_sim no)
@@
 		(on_board yes)
 		(dnp no)
-		(property "Reference" "#PWR053"
+		(property "Reference" "#PWR048"
 			(at 93.98 46.99 0)
 			(effects
@@
 			(project "openpcie2-rc-bplane"
 				(path "/4049bf06-3ac2-49e6-a199-57d4e4e4797e/6ab8d74d-40e9-45a1-a821-59a82de68ed7"
-					(reference "#PWR053")
+					(reference "#PWR048")
 					(unit 1)
 				)
@@
 		(on_board yes)
 		(dnp no)
-		(property "Reference" "#PWR056"
+		(property "Reference" "#PWR051"
 			(at 167.64 163.83 0)
 			(effects
@@
 			(project "openpcie2-rc-bplane"
 				(path "/4049bf06-3ac2-49e6-a199-57d4e4e4797e/6ab8d74d-40e9-45a1-a821-59a82de68ed7"
-					(reference "#PWR056")
+					(reference "#PWR051")
 					(unit 1)
 				)
@@
 		(on_board yes)
 		(dnp no)
-		(property "Reference" "#PWR050"
+		(property "Reference" "#PWR045"
 			(at 73.66 156.21 0)
 			(effects
@@
 			(project "openpcie2-rc-bplane"
 				(path "/4049bf06-3ac2-49e6-a199-57d4e4e4797e/6ab8d74d-40e9-45a1-a821-59a82de68ed7"
-					(reference "#PWR050")
+					(reference "#PWR045")
 					(unit 1)
 				)
@@
 		(on_board yes)
 		(dnp no)
-		(property "Reference" "R19"
+		(property "Reference" "R17"
 			(at 173.99 150.495 0)
 			(effects
@@
 			(project "openpcie2-rc-bplane"
 				(path "/4049bf06-3ac2-49e6-a199-57d4e4e4797e/6ab8d74d-40e9-45a1-a821-59a82de68ed7"
-					(reference "R19")
+					(reference "R17")
 					(unit 1)
 				)
@@
 		(on_board yes)
 		(dnp no)
-		(property "Reference" "#PWR058"
+		(property "Reference" "#PWR053"
 			(at 220.98 153.67 0)
 			(effects
@@
 			(project "openpcie2-rc-bplane"
 				(path "/4049bf06-3ac2-49e6-a199-57d4e4e4797e/6ab8d74d-40e9-45a1-a821-59a82de68ed7"
-					(reference "#PWR058")
+					(reference "#PWR053")
 					(unit 1)
 				)
@@
 		(on_board yes)
 		(dnp no)
-		(property "Reference" "R20"
+		(property "Reference" "R18"
 			(at 222.25 134.62 90)
 			(effects
@@
 			(project "openpcie2-rc-bplane"
 				(path "/4049bf06-3ac2-49e6-a199-57d4e4e4797e/6ab8d74d-40e9-45a1-a821-59a82de68ed7"
-					(reference "R20")
+					(reference "R18")
 					(unit 1)
 				)
@@
 		(on_board yes)
 		(dnp no)
-		(property "Reference" "#PWR057"
+		(property "Reference" "#PWR052"
 			(at 172.72 163.83 0)
 			(effects
@@
 			(project "openpcie2-rc-bplane"
 				(path "/4049bf06-3ac2-49e6-a199-57d4e4e4797e/6ab8d74d-40e9-45a1-a821-59a82de68ed7"
-					(reference "#PWR057")
+					(reference "#PWR052")
 					(unit 1)
 				)
@@
 		(on_board yes)
 		(dnp no)
-		(property "Reference" "R18"
+		(property "Reference" "R16"
 			(at 173.99 140.97 0)
 			(effects
@@
 			(project "openpcie2-rc-bplane"
 				(path "/4049bf06-3ac2-49e6-a199-57d4e4e4797e/6ab8d74d-40e9-45a1-a821-59a82de68ed7"
-					(reference "R18")
+					(reference "R16")
 					(unit 1)
 				)
@@
 		(on_board yes)
 		(dnp no)
-		(property "Reference" "R16"
+		(property "Reference" "R14"
 			(at 74.295 31.75 90)
 			(effects
@@
 			(project "openpcie2-rc-bplane"
 				(path "/4049bf06-3ac2-49e6-a199-57d4e4e4797e/6ab8d74d-40e9-45a1-a821-59a82de68ed7"
-					(reference "R16")
+					(reference "R14")
 					(unit 1)
 				)
@@
 		(on_board yes)
 		(dnp no)
-		(property "Reference" "R21"
+		(property "Reference" "R19"
 			(at 236.855 63.5 90)
 			(effects
@@
 			(project "openpcie2-rc-bplane"
 				(path "/4049bf06-3ac2-49e6-a199-57d4e4e4797e/6ab8d74d-40e9-45a1-a821-59a82de68ed7"
-					(reference "R21")
+					(reference "R19")
 					(unit 1)
 				)
@@
 			)
 		)
-		(property "DigiKey" "399-3683-1-ND"
+		(property "DigiKey" "PCE4579CT-ND"
 			(at 78.74 71.12 0)
 			(effects
@@
 			)
 		)
-		(property "Mouser" "80-T491A106K0067280"
+		(property "Mouser" "667-EEE-1CA101WAP"
 			(at 78.74 71.12 0)
 			(effects
@@
 			)
 		)
-		(property "TME" " T491A106K006AT"
+		(property "TME" "EEE1CA101WAP"
 			(at 78.74 71.12 0)
 			(effects
@@
 		(on_board yes)
 		(dnp no)
-		(property "Reference" "#PWR054"
+		(property "Reference" "#PWR049"
 			(at 121.92 148.59 0)
 			(effects
@@
 			(project "openpcie2-rc-bplane"
 				(path "/4049bf06-3ac2-49e6-a199-57d4e4e4797e/6ab8d74d-40e9-45a1-a821-59a82de68ed7"
-					(reference "#PWR054")
+					(reference "#PWR049")
 					(unit 1)
 				)
@@
 		(on_board yes)
 		(dnp no)
-		(property "Reference" "#PWR048"
+		(property "Reference" "#PWR043"
 			(at 48.26 29.21 0)
 			(effects
@@
 			(project "openpcie2-rc-bplane"
 				(path "/4049bf06-3ac2-49e6-a199-57d4e4e4797e/6ab8d74d-40e9-45a1-a821-59a82de68ed7"
-					(reference "#PWR048")
+					(reference "#PWR043")
 					(unit 1)
 				)
@@
 		(on_board yes)
 		(dnp no)
-		(property "Reference" "#PWR051"
+		(property "Reference" "#PWR046"
 			(at 78.74 82.55 0)
 			(effects
@@
 			(project "openpci2-backplane"
 				(path "/4049bf06-3ac2-49e6-a199-57d4e4e4797e/6ab8d74d-40e9-45a1-a821-59a82de68ed7"
-					(reference "#PWR051")
+					(reference "#PWR046")
 					(unit 1)
 				)
@@
 		(on_board yes)
 		(dnp no)
-		(property "Reference" "#PWR055"
+		(property "Reference" "#PWR050"
 			(at 139.7 161.29 0)
 			(effects
@@
 			(project "openpcie2-rc-bplane"
 				(path "/4049bf06-3ac2-49e6-a199-57d4e4e4797e/6ab8d74d-40e9-45a1-a821-59a82de68ed7"
-					(reference "#PWR055")
+					(reference "#PWR050")
 					(unit 1)
 				)
@@
 		(dnp no)
 		(fields_autoplaced yes)
-		(property "Reference" "#PWR059"
+		(property "Reference" "#PWR054"
 			(at 238.76 133.35 0)
 			(effects
@@
 			(project "openpcie2-rc-bplane"
 				(path "/4049bf06-3ac2-49e6-a199-57d4e4e4797e/6ab8d74d-40e9-45a1-a821-59a82de68ed7"
-					(reference "#PWR059")
+					(reference "#PWR054")
 					(unit 1)
 				)
@@
 		(on_board yes)
 		(dnp no)
-		(property "Reference" "#PWR060"
+		(property "Reference" "#PWR055"
 			(at 246.38 82.55 0)
 			(effects
@@
 			(project "openpcie2-rc-bplane"
 				(path "/4049bf06-3ac2-49e6-a199-57d4e4e4797e/6ab8d74d-40e9-45a1-a821-59a82de68ed7"
-					(reference "#PWR060")
+					(reference "#PWR055")
 					(unit 1)
 				)
@@
 		(on_board yes)
 		(dnp no)
-		(property "Reference" "#PWR046"
+		(property "Reference" "#PWR041"
 			(at 43.18 46.99 0)
 			(effects
@@
 			(project "openpcie2-rc-bplane"
 				(path "/4049bf06-3ac2-49e6-a199-57d4e4e4797e/6ab8d74d-40e9-45a1-a821-59a82de68ed7"
-					(reference "#PWR046")
+					(reference "#PWR041")
 					(unit 1)
 				)
@@
 		(on_board yes)
 		(dnp no)
-		(property "Reference" "U7"
+		(property "Reference" "U6"
 			(at 208.28 128.27 0)
 			(effects
@@
 			(project "openpcie2-rc-bplane"
 				(path "/4049bf06-3ac2-49e6-a199-57d4e4e4797e/6ab8d74d-40e9-45a1-a821-59a82de68ed7"
-					(reference "U7")
+					(reference "U6")
 					(unit 1)
 				)
@@
 		(on_board yes)
 		(dnp no)
-		(property "Reference" "#PWR052"
+		(property "Reference" "#PWR047"
 			(at 77.47 68.58 0)
 			(effects
@@
 			(project "openpcie2-rc-bplane"
 				(path "/4049bf06-3ac2-49e6-a199-57d4e4e4797e/6ab8d74d-40e9-45a1-a821-59a82de68ed7"
-					(reference "#PWR052")
+					(reference "#PWR047")
 					(unit 1)
 				)
@@
 		(on_board yes)
 		(dnp no)
-		(property "Reference" "#PWR047"
+		(property "Reference" "#PWR042"
 			(at 45.72 156.21 0)
 			(effects
@@
 			(project "openpcie2-rc-bplane"
 				(path "/4049bf06-3ac2-49e6-a199-57d4e4e4797e/6ab8d74d-40e9-45a1-a821-59a82de68ed7"
-					(reference "#PWR047")
+					(reference "#PWR042")
 					(unit 1)
 				)
@@
 		(on_board yes)
 		(dnp no)
-		(property "Reference" "#PWR049"
+		(property "Reference" "#PWR044"
 			(at 66.04 46.99 0)
 			(effects
@@
 			(project "openpcie2-rc-bplane"
 				(path "/4049bf06-3ac2-49e6-a199-57d4e4e4797e/6ab8d74d-40e9-45a1-a821-59a82de68ed7"
-					(reference "#PWR049")
+					(reference "#PWR044")
 					(unit 1)
 				)
@@
 		(on_board yes)
 		(dnp no)
-		(property "Reference" "R17"
+		(property "Reference" "R15"
 			(at 120.65 103.505 0)
 			(effects
@@
 			(project "openpcie2-rc-bplane"
 				(path "/4049bf06-3ac2-49e6-a199-57d4e4e4797e/6ab8d74d-40e9-45a1-a821-59a82de68ed7"
-					(reference "R17")
+					(reference "R15")
 					(unit 1)
 				)
@@
 			)
 		)
-		(property "Uvitron" "n/a"
-			(at 43.18 35.56 0)
-			(effects
-				(font
-					(size 1.27 1.27)
-				)
-				(hide yes)
-			)
-		)
 		(property "DigiKey" "SMBJ24ALFTR-ND"
 			(at 43.18 35.56 0)
@@
 			)
 		)
-		(property "Value" "~"
+		(property "Value" "n/a"
 			(at 114.3 129.54 0)
 			(effects

Commit message: Schematics update
Parts:
- added C51, C56: 100n, PCM_EEZ_passives:C_0603_1608Metric, symbol PCM_EEZ_passives:C-EU
- renumbered C48 to C49, C49 to C50, C50 to C52, C51 to C53, C52 to C54, C53 to C55, C54 to C57, C55 to C58, C56 to C59, C57 to C60, C58 to C61, C59 to C62, C60 to C63, C61 to C64, U6 to U7
Connections:
- net RC_RX0_N: now also J3.47 (PETn0/SATA-A-)
- net RC_RX0_P: now also J3.49 (PETp0/SATA-A+)
- net RC_TX0_N: now also C56.1
- net RC_TX0_P: now also C51.1
- net at J3.41 (PERn0/SATA-B+): now also C56.2
- net at J3.43 (PERp0/SATA-B-): now also C51.2
Other:
- note added: "Use it as main +3V3 rail?"
- note removed: "Enable in other way?"

Commit message: PCIe connectors update
Other:
- note added: "Connect to 3.3V?"
- moved on the sheet: C49, J2
