File: 1.pcb/openpci2-backplane/_autosave-clock_gen.kicad_sch (KiCad schematic)
At the start: 85 parts, among them J1 39-28-1063, J3 73251-3140, SW1 PTS645SK50SMTR92 LFS, U1 74LVC1G07GV,125, U2 TPS54KC23RZRR, U3 NCV308SNADJT1G, U4 SN74LVC244APWR, U5 TLV75801PDBVR, U6 PI6CG18801ZLIEX, Y1 TSX-3225 25.0000MF20X-AJ0

Commit message: Added extra Cout for buck istead of Cff
Parts:
- renumbered C101 to C16, C16 to C17, C17 to C18, C18 to C19, C19 to C20, C20 to C21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
