File: 1.pcb/openpci2-backplane/backplane.kicad_sch (KiCad schematic)
At the start: 13 parts, among them J10 10018784-10210TLF, J3 1-2199230-6, J4 1-2199230-6, J5 10018784-10210TLF, J6 1-2199230-6, J7 1-2199230-6, J8 10018784-10210TLF, J9 10018784-10210TLF

Commit message: SCH and PCB updates in prep for volume production and CrowdSupply campaign
Parts:
- D2: value ~ -> (none)
