File: 1.pcb/openpci2-backplane/openpci2-backplane.kicad_sch (KiCad schematic)
At the start: 19 parts

Commit message: SCH and PCB updates in prep for volume production and CrowdSupply campaign
Parts:
- FM1, FM2, FM3, FM4: value ~ -> (none)
- H1, H2, H3, H4, H5, H6: value Nylon Standoff M3x11 -> MountingHole
- H10, H11, H12, H7, H8, H9: value Nylon Screw M3x6 -> MountingHole; footprint (none) -> PCM_EEZ_THT:Mounting_hole 3.2_5.5mm_NO_NET
- LOGO3: footprint PCM_av_lib:PCIE2 logo -> PCM_Chili-chips:PCIE2 logo
Other:
- company: COPYRIGHT (C) Chili.CHIPS.ba doo -> COPYRIGHT (C) CHILI.CHIPS.LLC
- title: (none) -> openPCIE2 Backplane

Commit message: Cleanup in prep for the first release
Parts:
- H1, H2, H3, H4, H5, H6: value MountingHole -> Nylon Standoff M3x11; MPN (none) -> HP-11M3*11
Changed lines of the file:
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@@
 			)
 		)
-		(property "Value" "MountingHole"
+		(property "Value" "Nylon Standoff M3x11"
 			(at 168.91 187.9599 0)
 			(hide yes)
@@
 		)
 		(property "Datasheet" ""
+			(at 166.37 186.69 0)
+			(hide yes)
+			(show_name no)
+			(do_not_autoplace no)
+			(effects
+				(font
+					(size 1.27 1.27)
+				)
+			)
+		)
+		(property "MPN" "HP-11M3*11"
 			(at 166.37 186.69 0)
 			(hide yes)
@@
 			)
 		)
-		(property "Value" "MountingHole"
+		(property "Value" "Nylon Standoff M3x11"
 			(at 148.59 187.9599 0)
 			(hide yes)
@@
 		)
 		(property "Datasheet" ""
+			(at 146.05 186.69 0)
+			(hide yes)
+			(show_name no)
+			(do_not_autoplace no)
+			(effects
+				(font
+					(size 1.27 1.27)
+				)
+			)
+		)
+		(property "MPN" "HP-11M3*11"
 			(at 146.05 186.69 0)
 			(hide yes)
@@
 			)
 		)
-		(property "Value" "MountingHole"
+		(property "Value" "Nylon Standoff M3x11"
 			(at 118.11 187.9599 0)
 			(hide yes)
@@
 		)
 		(property "Datasheet" ""
+			(at 115.57 186.69 0)
+			(hide yes)
+			(show_name no)
+			(do_not_autoplace no)
+			(effects
+				(font
+					(size 1.27 1.27)
+				)
+			)
+		)
+		(property "MPN" "HP-11M3*11"
 			(at 115.57 186.69 0)
 			(hide yes)
@@
 			)
 		)
-		(property "Value" "MountingHole"
+		(property "Value" "Nylon Standoff M3x11"
 			(at 128.27 187.9599 0)
 			(hide yes)
@@
 		)
 		(property "Datasheet" ""
+			(at 125.73 186.69 0)
+			(hide yes)
+			(show_name no)
+			(do_not_autoplace no)
+			(effects
+				(font
+					(size 1.27 1.27)
+				)
+			)
+		)
+		(property "MPN" "HP-11M3*11"
 			(at 125.73 186.69 0)
 			(hide yes)
@@
 			)
 		)
-		(property "Value" "MountingHole"
+		(property "Value" "Nylon Standoff M3x11"
 			(at 158.75 187.9599 0)
 			(hide yes)
@@
 		)
 		(property "Datasheet" ""
+			(at 156.21 186.69 0)
+			(hide yes)
+			(show_name no)
+			(do_not_autoplace no)
+			(effects
+				(font
+					(size 1.27 1.27)
+				)
+			)
+		)
+		(property "MPN" "HP-11M3*11"
 			(at 156.21 186.69 0)
 			(hide yes)
@@
 			)
 		)
-		(property "Value" "MountingHole"
+		(property "Value" "Nylon Standoff M3x11"
 			(at 138.43 187.9599 0)
 			(hide yes)
@@
 			(at 135.89 186.69 0)
 			(hide yes)
+			(show_name no)
+			(do_not_autoplace no)
+			(effects
+				(font
+					(size 1.27 1.27)
+				)
+			)
+		)
+		(property "MPN" "HP-11M3*11"
+			(at 135.89 186.69 0)
+			(hide yes)

Commit message: cleaned up and aligned licensing info with project goal
Parts:
- H1, H2, H3, H4, H5, H6: LCSC C123698 -> (none)
- H10, H11, H12, H7, H8, H9: LCSC C194618 -> (none)
Changed lines of the file:
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@@
-			)
-		)
-		(property "LCSC" "C123698"
-			(at 166.37 186.69 0)
-			(hide yes)
-			(show_name no)
-			(do_not_autoplace no)
-			(effects
-				(font
-					(size 1.27 1.27)
-				)
 			)
 		)
@@
 			)
 		)
-		(property "DigiKey" ""
-			(at 36.83 189.23 0)
-			(hide yes)
-			(show_name no)
-			(do_not_autoplace no)
-			(effects
-				(font
-					(size 1.27 1.27)
-				)
-			)
-		)
 		(instances
 			(project "openpci2-backplane"
@@
 			)
 		)
-		(property "LCSC" "C194618"
-			(at 156.21 191.77 0)
-			(hide yes)
-			(show_name no)
-			(do_not_autoplace no)
-			(effects
-				(font
-					(size 1.27 1.27)
-				)
-			)
-		)
 		(instances
 			(project "openpci2-backplane"
@@
 			)
 		)
-		(property "LCSC" "C194618"
-			(at 146.05 191.77 0)
-			(hide yes)
-			(show_name no)
-			(do_not_autoplace no)
-			(effects
-				(font
-					(size 1.27 1.27)
-				)
-			)
-		)
 		(instances
 			(project "openpci2-backplane"
@@
 			)
 		)
-		(property "LCSC" "C123698"
-			(at 146.05 186.69 0)
-			(hide yes)
-			(show_name no)
-			(do_not_autoplace no)
-			(effects
-				(font
-					(size 1.27 1.27)
-				)
-			)
-		)
 		(instances
 			(project "openpci2-backplane"
@@
 			)
 		)
-		(property "DigiKey" ""
-			(at 26.67 189.23 0)
-			(hide yes)
-			(show_name no)
-			(do_not_autoplace no)
-			(effects
-				(font
-					(size 1.27 1.27)
-				)
-			)
-		)
 		(instances
 			(project "openpci2-backplane"
@@
 			)
 		)
-		(property "LCSC" "C123698"
-			(at 115.57 186.69 0)
-			(hide yes)
-			(show_name no)
-			(do_not_autoplace no)
-			(effects
-				(font
-					(size 1.27 1.27)
-				)
-			)
-		)
 		(instances
 			(project "openpci2-backplane"
@@
 			)
 		)
-		(property "LCSC" "C123698"
-			(at 125.73 186.69 0)
-			(hide yes)
-			(show_name no)
-			(do_not_autoplace no)
-			(effects
-				(font
-					(size 1.27 1.27)
-				)
-			)
-		)
 		(instances
 			(project "openpci2-backplane"
@@
 			)
 		)
-		(property "DigiKey" ""
-			(at 57.15 189.23 0)
-			(hide yes)
-			(show_name no)
-			(do_not_autoplace no)
-			(effects
-				(font
-					(size 1.27 1.27)
-				)
-			)
-		)
 		(instances
 			(project "openpci2-backplane"
@@
 			)
 		)
-		(property "LCSC" "C123698"
-			(at 156.21 186.69 0)
-			(hide yes)
-			(show_name no)
-			(do_not_autoplace no)
-			(effects
-				(font
-					(size 1.27 1.27)
-				)
-			)
-		)
 		(instances
 			(project "openpci2-backplane"
@@
 			)
 		)
-		(property "DigiKey" ""
-			(at 241.3 170.18 0)
-			(hide yes)
-			(show_name no)
-			(do_not_autoplace no)
-			(effects
-				(font
-					(size 1.27 1.27)
-				)
-			)
-		)
-		(property "LCSC" ""
-			(at 241.3 170.18 0)
-			(hide yes)
-			(show_name no)
-			(do_not_autoplace no)
-			(effects
-				(font
-					(size 1.27 1.27)
-				)
-			)
-		)
 		(instances
 			(project "openpci2-backplane"
@@
 			)
 		)
-		(property "LCSC" "C194618"
-			(at 115.57 191.77 0)
-			(hide yes)
-			(show_name no)
-			(do_not_autoplace no)
-			(effects
-				(font
-					(size 1.27 1.27)
-				)
-			)
-		)
 		(instances
 			(project "openpci2-backplane"
@@
 			)
 		)
-		(property "LCSC" "C194618"
-			(at 166.37 191.77 0)
-			(hide yes)
-			(show_name no)
-			(do_not_autoplace no)
-			(effects
-				(font
-					(size 1.27 1.27)
-				)
-			)
-		)
 		(instances
 			(project "openpci2-backplane"
@@
 			)
 		)
-		(property "LCSC" "C194618"
-			(at 125.73 191.77 0)
-			(hide yes)
-			(show_name no)
-			(do_not_autoplace no)
-			(effects
-				(font
-					(size 1.27 1.27)
-				)
-			)
-		)
 		(instances
 			(project "openpci2-backplane"
@@
 			)
 		)
-		(property "LCSC" "C194618"
-			(at 135.89 191.77 0)
-			(hide yes)
-			(show_name no)
-			(do_not_autoplace no)
-			(effects
-				(font
-					(size 1.27 1.27)
-				)
-			)
-		)
 		(instances
 			(project "openpci2-backplane"
@@
 			)
 		)
-		(property "LCSC" "C123698"
-			(at 135.89 186.69 0)
-			(hide yes)
-			(show_name no)
-			(do_not_autoplace no)
-			(effects
-				(font
-					(size 1.27 1.27)
-				)
-			)
-		)
 		(instances
 			(project "openpci2-backplane"
@@
 			(at 46.99 189.23 0)
 			(hide yes)
-			(show_name no)
-			(do_not_autoplace no)
-			(effects
-				(font
-					(size 1.27 1.27)
-				)
-			)
-		)
-		(property "DigiKey" ""
-			(at 46.99 189.23 0)
-			(hide yes)

Commit message: cont'd cleanup in prep for a first official release
Parts:
- H10, H11, H12, H7, H8, H9: now left out of the parts list
Changed lines of the file:
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@@
 	(title_block
 		(title "openPCIE2 Backplane")
-		(date "2026-09-08")
-		(rev "r1B1")
+		(date "2026-10-06")
+		(rev "RevB")
 		(company "COPYRIGHT (C) CHILI.CHIPS.LLC")
 		(comment 1 "https://cern-ohl.web.cern.ch")
@@
 		(body_style 1)
 		(exclude_from_sim no)
-		(in_bom yes)
+		(in_bom no)
 		(on_board no)
 		(in_pos_files yes)
@@
 		(body_style 1)
 		(exclude_from_sim no)
-		(in_bom yes)
+		(in_bom no)
 		(on_board no)
 		(in_pos_files yes)
@@
 		(body_style 1)
 		(exclude_from_sim no)
-		(in_bom yes)
+		(in_bom no)
 		(on_board no)
 		(in_pos_files yes)
@@
 		(body_style 1)
 		(exclude_from_sim no)
-		(in_bom yes)
+		(in_bom no)
 		(on_board no)
 		(in_pos_files yes)
@@
 		(body_style 1)
 		(exclude_from_sim no)
-		(in_bom yes)
+		(in_bom no)
 		(on_board no)
 		(in_pos_files yes)
@@
 		(body_style 1)
 		(exclude_from_sim no)
-		(in_bom yes)
+		(in_bom no)
 		(on_board no)
 		(in_pos_files yes)
